File: 02_entrada.kicad_sch (KiCad schematic)
At the start: 9 parts, among them T1 TP_+24V, T2 TP_GND_ADC_P1

Commit message: Esquematico: alimentacao do lado PLC passa da folha 3 para a folha 4
U2 (MCP1824, +3.3V do lado DGND), C6, C8, C9, T3 e T5 desenhados na
folha 4 (barreira digital), junto ao ISO7141 que alimentam. Limpeza
grafica nas folhas 2 e 6 (rectangulos e fios soltos).

Sem mudanca electrica: netlist com os mesmos 148 componentes e nenhum
pino com rede diferente; ERC 0 erros; DRC 0 erros, paridade 0.

Co-Authored-By: Claude Opus 5.5 (1M context) <noreply@anthropic.com>
Changed lines of the file:
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@@
-	)
-	(junction
-		(at 69.85 165.1)
-		(diameter 0)
-		(color 0 0 0 0)
 	)
 	(junction
@@
 		(diameter 0)
 		(color 0 0 0 0)
-	)
-	(junction
-		(at 88.9 165.1)
-		(diameter 0)
-		(color 0 0 0 0)
