File: 06_lacos.kicad_sch (KiCad schematic)
At the start: 58 parts, among them T8 TP_+24V_ADC, U10 TPS26613DDFR, U11 TPS26613DDFR, U12 TPS7A4001DGN, U8 TPS26613DDFR, U9 TPS26613DDFR

Commit message: Esquematico: alimentacao do lado PLC passa da folha 3 para a folha 4
U2 (MCP1824, +3.3V do lado DGND), C6, C8, C9, T3 e T5 desenhados na
folha 4 (barreira digital), junto ao ISO7141 que alimentam. Limpeza
grafica nas folhas 2 e 6 (rectangulos e fios soltos).

Sem mudanca electrica: netlist com os mesmos 148 componentes e nenhum
pino com rede diferente; ERC 0 erros; DRC 0 erros, paridade 0.

Co-Authored-By: Claude Opus 5.5 (1M context) <noreply@anthropic.com>
Changed lines of the file:
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@@
 	)
 	(rectangle
-		(start 208.28 109.22)
-		(end 265.43 134.62)
-		(stroke
-			(width 0)
-			(type default)
-		)
-		(fill
-			(type none)
-		)
-	)
-	(rectangle
-		(start 208.28 143.51)
-		(end 265.43 168.91)
-		(stroke
-			(width 0)
-			(type default)
-		)
-		(fill
-			(type none)
-		)
-	)
-	(rectangle
 		(start 208.28 179.07)
 		(end 265.43 204.47)
@@
 		)
 	)
-	(rectangle
-		(start 208.28 77.47)
-		(end 265.43 102.87)
-		(stroke
-			(width 0)
-			(type default)
-		)
-		(fill
-			(type none)
-		)
-	)
 	(text "    o 1 uF de entrada vem do C4 (10 uF 100 V, ~6 uF a 24 V) no"
 		(exclude_from_sim no)
@@
 	(wire
 		(pts
-			(xy 49.53 33.02) (xy 49.53 31.75)
-		)
-		(stroke
-			(width 0)
-			(type default)
-		)
-	)
-	(wire
-		(pts
 			(xy 233.68 69.85) (xy 236.22 69.85)
 		)
@@
 	(wire
 		(pts
-			(xy 49.53 33.02) (xy 55.88 33.02)
-		)
-		(stroke
-			(width 0)
-			(type default)
-		)
-	)
-	(wire
-		(pts
 			(xy 67.31 64.77) (xy 74.93 64.77)
 		)
@@
 	(symbol
 		(lib_id "power:+5V")
-		(at 49.53 31.75 0)
+		(at 55.88 33.02 0)
 		(unit 1)
 		(body_style 1)
@@
 		(dnp no)
 		(property "Reference" "#PWR086"
-			(at 49.53 38.1 0)
+			(at 55.88 39.37 0)
 			(hide yes)
 			(show_name no)
@@
 		)
 		(property "Value" "+12V_TPS"
-			(at 50.8 26.67 0)
+			(at 57.15 27.94 0)
 			(show_name no)
 			(do_not_autoplace no)
@@
 		)
 		(property "Footprint" ""
-			(at 49.53 31.75 0)
+			(at 55.88 33.02 0)
 			(hide yes)
 			(show_name no)
@@
 		)
 		(property "Datasheet" ""
-			(at 49.53 31.75 0)
+			(at 55.88 33.02 0)
 			(hide yes)
 			(show_name no)
@@
 		)
 		(property "Description" ""
-			(at 49.53 31.75 0)
+			(at 55.88 33.02 0)
 			(show_name no)
 			(do_not_autoplace no)
