File: Desenvolvimento_IC2S-EBM7-2608-V2.3-Fixo420/Projeto_IC2S-EBM7-2608-V2.3-Fixo420/03_alimentacao.kicad_sch (KiCad schematic)
At the start: 23 parts, among them T4 TP_+5V_REG, T6 TP_+3.3V_ANA, U1 R-78HB5.0-0.5L, U3 SPX3819M5-L-3-3/TR, U4 TL431B

Commit message: Revisao da reuniao 28-09: ramo unico de 24 V, 100 nF a 50 V, um so MPN de 1 uF
- Saem F2, o diodo e o condensador do ramo +24V_ADC; F1 + diodo alimentam o
  R-78HB e o +24V_ADC. +24V_REG deixa de existir (esquematico, PCB, netclasses).
- Condensador de entrada do R-78HB conferido contra o datasheet Recom (p.4):
  10 uF/100 V cumpre os 3,3 uF/100 V pedidos com Vin > 50 V. Sem alteracao.
- 100 nF fora do 24 V -> TDK C1608X7R1H104K080AA (50 V); o do +24V_ADC fica
  GRM188R72A104KA35D (100 V). 1 uF -> TDK C1608X7R1H105K080AB nos quatro.
- Notas 2, 13 e 14 da folha 2; README e registo em 00-Especificacoes;
  catalogo TDK em Documentos_de_Referencia.

Co-Authored-By: Claude Opus 5.5 (1M context) <noreply@anthropic.com>
Claude-Session: https://claude.ai/code/session_01KPnkiJQKrkjgRqqw9M78ie
Parts:
- C10, C12, C4: value 100nF -> 100nF/50V; MPN GRM188R72A104KA35D -> C1608X7R1H104K080AA
Connections:
- net +24V_REG renamed +24V_ADC
Other:
- note added: "1. Cadeia analogica: +24V_ADC > U3 K78U05 > +5V_REG >"
- note removed: "1. Cadeia analogica: +24V_REG > U3 K78U05 > +5V_REG >"
Changed lines of the file:
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@@
 		)
 	)
-	(text "1. Cadeia analogica: +24V_REG > U3 K78U05 > +5V_REG >"
+	(text "1. Cadeia analogica: +24V_ADC > U3 K78U05 > +5V_REG >"
 		(exclude_from_sim no)
 		(at 35.56 102.87 0)
@@
 			)
 		)
-		(property "Value" "100nF"
+		(property "Value" "100nF/50V"
 			(at 146.05 72.39 0)
 			(show_name no)
@@
 			)
 		)
-		(property "MPN" "GRM188R72A104KA35D"
+		(property "MPN" "C1608X7R1H104K080AA"
 			(at 0 0 0)
 			(hide yes)
@@
 			)
 		)
-		(property "Value" "100nF"
+		(property "Value" "100nF/50V"
 			(at 166.37 72.39 0)
 			(show_name no)
@@
 			)
 		)
-		(property "MPN" "GRM188R72A104KA35D"
+		(property "MPN" "C1608X7R1H104K080AA"
 			(at 0 0 0)
 			(hide yes)
@@
 			)
 		)
-		(property "Value" "100nF"
+		(property "Value" "100nF/50V"
 			(at 62.738 73.914 0)
 			(show_name no)
@@
 			)
 		)
-		(property "MPN" "GRM188R72A104KA35D"
+		(property "MPN" "C1608X7R1H104K080AA"
 			(at 0 0 0)
 			(hide yes)
@@
 			)
 		)
-		(property "Value" "+24V_REG"
+		(property "Value" "+24V_ADC"
 			(at 30.48 58.42 0)
 			(show_name no)
