File: Desenvolvimento_IC2S-EBM7-2608-V2.3-Fixo420/Projeto_IC2S-EBM7-2608-V2.3-Fixo420/05_adc.kicad_sch (KiCad schematic)
At the start: 17 parts, among them T7 TP_GND_ADC, U6 AD7124-8BCPZ, U7 ADR4525BRZ

Commit message: Revisao da reuniao 28-09: ramo unico de 24 V, 100 nF a 50 V, um so MPN de 1 uF
- Saem F2, o diodo e o condensador do ramo +24V_ADC; F1 + diodo alimentam o
  R-78HB e o +24V_ADC. +24V_REG deixa de existir (esquematico, PCB, netclasses).
- Condensador de entrada do R-78HB conferido contra o datasheet Recom (p.4):
  10 uF/100 V cumpre os 3,3 uF/100 V pedidos com Vin > 50 V. Sem alteracao.
- 100 nF fora do 24 V -> TDK C1608X7R1H104K080AA (50 V); o do +24V_ADC fica
  GRM188R72A104KA35D (100 V). 1 uF -> TDK C1608X7R1H105K080AB nos quatro.
- Notas 2, 13 e 14 da folha 2; README e registo em 00-Especificacoes;
  catalogo TDK em Documentos_de_Referencia.

Co-Authored-By: Claude Opus 5.5 (1M context) <noreply@anthropic.com>
Claude-Session: https://claude.ai/code/session_01KPnkiJQKrkjgRqqw9M78ie
Parts:
- C18, C19, C20, C23, C24: value 100nF -> 100nF/50V; MPN GRM188R72A104KA35D -> C1608X7R1H104K080AA
- C21: value 1uF -> 1uF/50V; MPN 885012206002 -> C1608X7R1H105K080AB
- C22: value 1uF -> 1uF/50V; MPN C0603C105K4RACTU -> C1608X7R1H105K080AB
Changed lines of the file:
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@@
 			)
 		)
-		(property "Value" "1uF"
+		(property "Value" "1uF/50V"
 			(at 182.88 89.154 0)
 			(show_name no)
@@
 			)
 		)
-		(property "MPN" "C0603C105K4RACTU"
+		(property "MPN" "C1608X7R1H105K080AB"
 			(at 0 0 0)
 			(hide yes)
@@
 			)
 		)
-		(property "Value" "100nF"
+		(property "Value" "100nF/50V"
 			(at 149.86 128.27 270)
 			(show_name no)
@@
 			)
 		)
-		(property "MPN" "GRM188R72A104KA35D"
+		(property "MPN" "C1608X7R1H104K080AA"
 			(at 0 10.16 0)
 			(hide yes)
@@
 			)
 		)
-		(property "Value" "100nF"
+		(property "Value" "100nF/50V"
 			(at 146.304 117.094 270)
 			(show_name no)
@@
 			)
 		)
-		(property "MPN" "GRM188R72A104KA35D"
+		(property "MPN" "C1608X7R1H104K080AA"
 			(at 0 -5.08 0)
 			(hide yes)
@@
 			)
 		)
-		(property "Value" "100nF"
+		(property "Value" "100nF/50V"
 			(at 198.882 88.646 0)
 			(show_name no)
@@
 			)
 		)
-		(property "MPN" "GRM188R72A104KA35D"
+		(property "MPN" "C1608X7R1H104K080AA"
 			(at 0 0 0)
 			(hide yes)
@@
 			)
 		)
-		(property "Value" "100nF"
+		(property "Value" "100nF/50V"
 			(at 220.472 88.392 0)
 			(show_name no)
@@
 			)
 		)
-		(property "MPN" "GRM188R72A104KA35D"
+		(property "MPN" "C1608X7R1H104K080AA"
 			(at 0 0 0)
 			(hide yes)
@@
 			)
 		)
-		(property "Value" "100nF"
+		(property "Value" "100nF/50V"
 			(at 146.558 109.22 0)
 			(show_name no)
@@
 			)
 		)
-		(property "MPN" "GRM188R72A104KA35D"
+		(property "MPN" "C1608X7R1H104K080AA"
 			(at 0 0 0)
 			(hide yes)
@@
 			)
 		)
-		(property "Value" "1uF"
+		(property "Value" "1uF/50V"
 			(at 160.274 106.68 0)
 			(show_name no)
@@
 			)
 		)
-		(property "MPN" "885012206002"
+		(property "MPN" "C1608X7R1H105K080AB"
 			(at 0 0 0)
 			(hide yes)
