File: Desenvolvimento_IC2S-EBM7-2608-V2.3-Fixo420/Projeto_IC2S-EBM7-2608-V2.3-Fixo420/08_ntc.kicad_sch (KiCad schematic)
At the start: 5 parts

Commit message: NTC com simbolo de termistor e explicacao do TL431 do +3.3V_ANA
- Folha 8: o NTC deixa de usar Device:R e passa a Device:Thermistor_NTC
  (mesmos pinos; netlist e PCB inalterados). Observacao da reuniao de 25-09.
- Documento porque_TL431_*_no_3V3_ANA.md: o LDO nao absorve corrente, os
  BAV199 despejam os surtos no rail e o TL431 segura-o abaixo do maximo
  absoluto do AD7124; numeros tirados dos datasheets locais.

Co-Authored-By: Claude Opus 5.5 (1M context) <noreply@anthropic.com>
Claude-Session: https://claude.ai/code/session_01KPnkiJQKrkjgRqqw9M78ie
Parts:
- R36: symbol Device:R -> Device:Thermistor_NTC
Changed lines of the file:
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@@
 	)
 	(symbol
-		(lib_id "Device:R")
+		(lib_id "Device:Thermistor_NTC")
 		(at 41.91 58.42 0)
 		(unit 1)
