File: Desenvolvimento_IC2S-EBM7-2608-V2.3-Fixo420/Projeto_IC2S-EBM7-2608-V2.3-Fixo420/04_barreira.kicad_sch (KiCad schematic)
At the start: 8 parts, among them T3 TP_DGND, T5 TP_+3.3V_DIG, U2 SPX3819M5-L-3-3/TR, U5 ISO7141CCDBQR

Commit message: C49 2,2 uF na saida do U2 (SPX3819), como a saida do SPX da V2.2 em campo
- Datasheet SPX3819 Fig. 18 (p.8) conferido: EN a VIN e BYP aberto como a figura; saida
  cerâmica 2,2 + 10 uF + 100 nF (V2.2 so tinha ceramicos no SPX). MPN C1608X5R1E225K080AB
  ja na BOM (C7/C11/C46). PCB: clone do C8 a 3 mm do U2, 2 ligacoes por rotear.
- Inclui as alteracoes de roteamento em curso do projectista no PCB.
- ERC 0; DRC 0 erros, sem avisos novos, paridade 0. BOM e PDF regenerados.

Co-Authored-By: Claude Opus 5.5 (1M context) <noreply@anthropic.com>
Claude-Session: https://claude.ai/code/session_01KPnkiJQKrkjgRqqw9M78ie
Parts:
- added C49: 2.2uF, EBM7_V23:0603C, symbol Device:C
Connections:
- net +3.3V: now also C49.2
- net DGND: now also C49.1
Changed lines of the file:
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@@
 		(at 58.42 53.34)
+	)
+	(symbol
+		(lib_id "Device:C")
+		(at 86.36 58.42 180)
+		(unit 1)
+		(body_style 1)
+		(exclude_from_sim no)
+		(in_bom yes)
+		(on_board yes)
+		(in_pos_files yes)
+		(dnp no)
+		(property "Reference" "C49"
+			(at 90.8 56.52 0)
+			(show_name no)
+			(do_not_autoplace no)
+			(effects
+				(font
+					(size 1.27 1.27)
+				)
+			)
+		)
+		(property "Value" "2.2uF"
+			(at 90.8 59.05 0)
+			(show_name no)
+			(do_not_autoplace no)
+			(effects
+				(font
+					(size 1.27 1.27)
+				)
+			)
+		)
+		(property "Footprint" "EBM7_V23:0603C"
+			(at 86.36 58.42 180)
+			(hide yes)
+			(show_name no)
+			(do_not_autoplace no)
+			(effects
+				(font
+					(size 1.27 1.27)
+				)
+			)
+		)
+		(property "Datasheet" ""
+			(at 86.36 58.42 0)
+			(hide yes)
+			(show_name no)
+			(do_not_autoplace no)
+			(effects
+				(font
+					(size 1.27 1.27)
+				)
+			)
+		)
+		(property "Description" ""
+			(at 86.36 58.42 0)
+			(show_name no)
+			(do_not_autoplace no)
+			(effects
+				(font
+					(size 1.27 1.27)
+				)
+			)
+		)
+		(property "MPN" "C1608X5R1E225K080AB"
+			(at -27.94 -88.9 0)
+			(hide yes)
+			(show_name no)
+			(do_not_autoplace no)
+			(effects
+				(font
+					(size 1.27 1.27)
+				)
+			)
+		)
+		(pin "1"
+		)
+		(pin "2"
+		)
+		(instances
+			(project "IC2S-EBM7-2608-V2.3-Fixo420"
+				(path "/ea39faa7-2c85-4731-99b5-dc619370fd78/e9834b1b-d21f-47ea-ad01-85c539f0c334"
+					(reference "C49")
+					(unit 1)
+				)
+			)
+		)
+	)
+	(symbol
+		(lib_id "power:GND")
+		(at 86.36 62.23 0)
+		(unit 1)
+		(body_style 1)
+		(exclude_from_sim no)
+		(in_bom yes)
+		(on_board yes)
+		(in_pos_files yes)
+		(dnp no)
+		(property "Reference" "#PWR0153"
+			(at 86.36 55.88 0)
+			(hide yes)
+			(show_name no)
+			(do_not_autoplace no)
+			(effects
+				(font
+					(size 1.27 1.27)
+				)
+			)
+		)
+		(property "Value" "DGND"
+			(at 86.36 66.04 0)
+			(show_name no)
+			(do_not_autoplace no)
+			(effects
+				(font
+					(size 1.27 1.27)
+				)
+			)
+		)
+		(property "Footprint" ""
+			(at 86.36 62.23 0)
+			(hide yes)
+			(show_name no)
+			(do_not_autoplace no)
+			(effects
+				(font
+					(size 1.27 1.27)
+				)
+			)
+		)
+		(property "Datasheet" ""
+			(at 86.36 62.23 0)
+			(hide yes)
+			(show_name no)
+			(do_not_autoplace no)
+			(effects
+				(font
+					(size 1.27 1.27)
+				)
+			)
+		)
+		(property "Description" ""
+			(at 86.36 62.23 0)
+			(show_name no)
+			(do_not_autoplace no)
+			(effects
+				(font
+					(size 1.27 1.27)
+				)
+			)
+		)
+		(pin "1"
+		)
+		(instances
+			(project "IC2S-EBM7-2608-V2.3-Fixo420"
+				(path "/ea39faa7-2c85-4731-99b5-dc619370fd78/e9834b1b-d21f-47ea-ad01-85c539f0c334"
+					(reference "#PWR0153")
+					(unit 1)
+				)
+			)
+		)
+	)
+	(symbol
+		(lib_id "power:+3V3")
+		(at 86.36 54.61 0)
+		(unit 1)
+		(body_style 1)
+		(exclude_from_sim no)
+		(in_bom yes)
+		(on_board yes)
+		(in_pos_files yes)
+		(dnp no)
+		(property "Reference" "#PWR0154"
+			(at 86.36 48.26 0)
+			(hide yes)
+			(show_name no)
+			(do_not_autoplace no)
+			(effects
+				(font
+					(size 1.27 1.27)
+				)
+			)
+		)
+		(property "Value" "+3.3V"
+			(at 86.36 49.53 0)
+			(show_name no)
+			(do_not_autoplace no)
+			(effects
+				(font
+					(size 1.27 1.27)
+				)
+			)
+		)
+		(property "Footprint" ""
+			(at 86.36 54.61 0)
+			(hide yes)
+			(show_name no)
+			(do_not_autoplace no)
+			(effects
+				(font
+					(size 1.27 1.27)
+				)
+			)
+		)
+		(property "Datasheet" ""
+			(at 86.36 54.61 0)
+			(hide yes)
+			(show_name no)
+			(do_not_autoplace no)
+			(effects
+				(font
+					(size 1.27 1.27)
+				)
+			)
+		)
+		(property "Description" ""
+			(at 86.36 54.61 0)
+			(show_name no)
+			(do_not_autoplace no)
+			(effects
+				(font
+					(size 1.27 1.27)
+				)
+			)
+		)
+		(pin "1"
+		)
+		(instances
+			(project "IC2S-EBM7-2608-V2.3-Fixo420"
+				(path "/ea39faa7-2c85-4731-99b5-dc619370fd78/e9834b1b-d21f-47ea-ad01-85c539f0c334"
+					(reference "#PWR0154")
+					(unit 1)
+				)
+			)
+		)
 	)
 	(sheet_instances
