File: Desenvolvimento_IC2S-EBM7-2608-V2.3-Fixo420/Projeto_IC2S-EBM7-2608-V2.3-Fixo420/02_entrada.kicad_sch (KiCad schematic)
At the start: 6 parts, among them T1 TP_+24V, T2 TP_GND_ADC_P1

Commit message: Roteamento do U2 (SPX3819) e do bypass do ISO7141; pacote de fabricacao regenerado
PCB:
- C49 (2,2 uF) e C8 (10 uF) junto do VOUT do U2 (1,68 e 2,23 mm), C6 na
  entrada a 3,0 mm.
- C9 (100 nF) reposto como bypass do VCC1 do U5 (1,93 mm), massa por via
  DGND a 1,0 mm do pad. Tinha sido movido com o grupo do U2 (6,3 mm).
- Rede unconnected-(U2-BP-Pad4) na classe DIGSIDE (pad NC do SPX3819 dentro
  da zona DGND; sem isto a regra de barreira de 1,0 mm disparava contra C9).
- DRC kicad-cli com paridade: 0 erros, 0 avisos, 0 desligados, paridade 0.

Esquematico: sem alteracao electrica (paridade 0, netlist igual). Restauro do
historico local do KiCad: coordenadas arredondadas (02), fios colineares
fundidos com os mesmos extremos (04), rectangulo grafico removido (06),
ordem dos textos (08).

Fabricacao: Gerbers, furacao, PnP, stencil, BOM, vistas, STEP e PDF do
esquematico regenerados desta placa (antes eram de 28-09 02:48).

Co-Authored-By: Claude Opus 5.5 (1M context) <noreply@anthropic.com>
Claude-Session: https://claude.ai/code/session_01KPnkiJQKrkjgRqqw9M78ie
Changed lines of the file:
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@@
+		)
+	)
+	(text "13. RAMO UNICO DE 24 V (reuniao da equipa, 2026-09-28):"
+		(exclude_from_sim no)
+		(at 22.86 83.82 0)
+		(effects
+			(font
+				(size 1.27 1.27)
+			)
+			(justify left bottom)
+		)
+	)
+	(text "    Pior caso fora do 24 V: +12V_TPS a 31,7 V (folha 6,"
+		(exclude_from_sim no)
+		(at 22.86 137.16 0)
+		(effects
+			(font
+				(size 1.27 1.27)
+			)
+			(justify left bottom)
 		)
 	)
@@
 		)
 	)
+	(text "    Arranque ~30 uF: ~5 mA2s (escala da nota 10) contra"
+		(exclude_from_sim no)
+		(at 22.86 106.68 0)
+		(effects
+			(font
+				(size 1.27 1.27)
+			)
+			(justify left bottom)
+		)
+	)
+	(text "    F1 750 mA e D2 MBR1H100SF 1 A chegam."
+		(exclude_from_sim no)
+		(at 22.86 102.87 0)
+		(effects
+			(font
+				(size 1.27 1.27)
+			)
+			(justify left bottom)
+		)
+	)
+	(text "    Perde-se a selectividade: curto no +24V_ADC abre F1."
+		(exclude_from_sim no)
+		(at 22.86 114.3 0)
+		(effects
+			(font
+				(size 1.27 1.27)
+			)
+			(justify left bottom)
+		)
+	)
 	(text "   MLCC de 50 V - mecanismo A. Peca exata por escolher."
 		(exclude_from_sim no)
@@
 		)
 	)
+	(text "    1 uF = TDK C1608X7R1H105K080AB (X7R 50 V, p.35) nos 4."
+		(exclude_from_sim no)
+		(at 22.86 148.59 0)
+		(effects
+			(font
+				(size 1.27 1.27)
+			)
+			(justify left bottom)
+		)
+	)
+	(text "    150 mA2s do CC12H750MA, ~29x de margem."
+		(exclude_from_sim no)
+		(at 22.86 110.49 0)
+		(effects
+			(font
+				(size 1.27 1.27)
+			)
+			(justify left bottom)
+		)
+	)
 	(text "4. C1/C13 = 10 uF a 100 V: o clamp de 53,3 V fica acima de"
 		(exclude_from_sim no)
@@
 		)
 	)
+	(text "    TDK C1608X7R1H104K080AA (X7R 50 V, catalogo TDK p.34)."
+		(exclude_from_sim no)
+		(at 22.86 133.35 0)
+		(effects
+			(font
+				(size 1.27 1.27)
+			)
+			(justify left bottom)
+		)
+	)
 	(text "    de GND_ADC (era GND_24V). Escolha do projectista 2026-09-04."
 		(exclude_from_sim no)
@@
 		)
 	)
+	(text "    saem F2, D3 e C2. Tudo vem dos mesmos 24 V: nao eram"
+		(exclude_from_sim no)
+		(at 22.86 87.63 0)
+		(effects
+			(font
+				(size 1.27 1.27)
+			)
+			(justify left bottom)
+		)
+	)
+	(text "    116 mA em regime, ~180 mA em falha (folha 1, nota 2):"
+		(exclude_from_sim no)
+		(at 22.86 99.06 0)
+		(effects
+			(font
+				(size 1.27 1.27)
+			)
+			(justify left bottom)
+		)
+	)
 	(text "   ponto unico de uniao das terras (R200/R1, removido - nota 7)."
 		(exclude_from_sim no)
@@
 		)
 	)
+	(text "    nota 17), por isso 50 V e nao 25 V. C36 (+24V_ADC,"
+		(exclude_from_sim no)
+		(at 22.86 140.97 0)
+		(effects
+			(font
+				(size 1.27 1.27)
+			)
+			(justify left bottom)
+		)
+	)
 	(text "3. D200 = SMA6J33A-Q (Bourns): VRWM 33 V, VBR 36,7-40,6 V,"
 		(exclude_from_sim no)
@@
 		)
 	)
+	(text "    ate 53,3 V) fica GRM188R72A104KA35D 100 V."
+		(exclude_from_sim no)
+		(at 22.86 144.78 0)
+		(effects
+			(font
+				(size 1.27 1.27)
+			)
+			(justify left bottom)
+		)
+	)
+	(text "    o U1 (R-78HB) e o +24V_ADC; +24V_REG deixa de existir."
+		(exclude_from_sim no)
+		(at 22.86 95.25 0)
+		(effects
+			(font
+				(size 1.27 1.27)
+			)
+			(justify left bottom)
+		)
+	)
 	(text "    10 uF/100 V ceramico junto ao Vin (C13); C1 e o bulk"
 		(exclude_from_sim no)
@@
 		)
 	)
+	(text "14. CONDENSADORES (2026-09-28): 100 nF fora do 24 V ="
+		(exclude_from_sim no)
+		(at 22.86 129.54 0)
+		(effects
+			(font
+				(size 1.27 1.27)
+			)
+			(justify left bottom)
+		)
+	)
+	(text "    canais independentes nem isolados. F1 + D2 alimentam"
+		(exclude_from_sim no)
+		(at 22.86 91.44 0)
+		(effects
+			(font
+				(size 1.27 1.27)
+			)
+			(justify left bottom)
+		)
+	)
 	(text "1. F1 = CC12H750MA-TR (Eaton, time-lag). I2t de fusao 150 mA2s,"
 		(exclude_from_sim no)
@@
 		)
 	)
+	(text "    3,3 uF/100 V se Vin > 50 V (clamp 53,3 V): 10 uF cumpre."
+		(exclude_from_sim no)
+		(at 22.86 121.92 0)
+		(effects
+			(font
+				(size 1.27 1.27)
+			)
+			(justify left bottom)
+		)
+	)
 	(text "    (os cortos de campo param no TPS26613 e em F3-F6). 100 mA em"
 		(exclude_from_sim no)
@@
 		(exclude_from_sim no)
 		(at 114.3 160.02 0)
+		(effects
+			(font
+				(size 1.27 1.27)
+			)
+			(justify left bottom)
+		)
+	)
+	(text "    C1 = entrada do R-78HB: Recom R-78HB-0.5 p.4 pede"
+		(exclude_from_sim no)
+		(at 22.86 118.11 0)
 		(effects
 			(font
@@
 		)
 	)
-	(text "13. RAMO UNICO DE 24 V (reuniao da equipa, 2026-09-28):"
-		(exclude_from_sim no)
-		(at 22.86 83.82 0)
-		(effects
-			(font
-				(size 1.27 1.27)
-			)
-			(justify left bottom)
-		)
-	)
-	(text "    saem F2, D3 e C2. Tudo vem dos mesmos 24 V: nao eram"
-		(exclude_from_sim no)
-		(at 22.86 87.63 0)
-		(effects
-			(font
-				(size 1.27 1.27)
-			)
-			(justify left bottom)
-		)
-	)
-	(text "    canais independentes nem isolados. F1 + D2 alimentam"
-		(exclude_from_sim no)
-		(at 22.86 91.44 0)
-		(effects
-			(font
-				(size 1.27 1.27)
-			)
-			(justify left bottom)
-		)
-	)
-	(text "    o U1 (R-78HB) e o +24V_ADC; +24V_REG deixa de existir."
-		(exclude_from_sim no)
-		(at 22.86 95.25 0)
-		(effects
-			(font
-				(size 1.27 1.27)
-			)
-			(justify left bottom)
-		)
-	)
-	(text "    116 mA em regime, ~180 mA em falha (folha 1, nota 2):"
-		(exclude_from_sim no)
-		(at 22.86 99.05999999999999 0)
-		(effects
-			(font
-				(size 1.27 1.27)
-			)
-			(justify left bottom)
-		)
-	)
-	(text "    F1 750 mA e D2 MBR1H100SF 1 A chegam."
-		(exclude_from_sim no)
-		(at 22.86 102.86999999999999 0)
-		(effects
-			(font
-				(size 1.27 1.27)
-			)
-			(justify left bottom)
-		)
-	)
-	(text "    Arranque ~30 uF: ~5 mA2s (escala da nota 10) contra"
-		(exclude_from_sim no)
-		(at 22.86 106.67999999999999 0)
-		(effects
-			(font
-				(size 1.27 1.27)
-			)
-			(justify left bottom)
-		)
-	)
-	(text "    150 mA2s do CC12H750MA, ~29x de margem."
-		(exclude_from_sim no)
-		(at 22.86 110.49 0)
-		(effects
-			(font
-				(size 1.27 1.27)
-			)
-			(justify left bottom)
-		)
-	)
-	(text "    Perde-se a selectividade: curto no +24V_ADC abre F1."
-		(exclude_from_sim no)
-		(at 22.86 114.3 0)
-		(effects
-			(font
-				(size 1.27 1.27)
-			)
-			(justify left bottom)
-		)
-	)
-	(text "    C1 = entrada do R-78HB: Recom R-78HB-0.5 p.4 pede"
-		(exclude_from_sim no)
-		(at 22.86 118.10999999999999 0)
-		(effects
-			(font
-				(size 1.27 1.27)
-			)
-			(justify left bottom)
-		)
-	)
-	(text "    3,3 uF/100 V se Vin > 50 V (clamp 53,3 V): 10 uF cumpre."
-		(exclude_from_sim no)
-		(at 22.86 121.91999999999999 0)
-		(effects
-			(font
-				(size 1.27 1.27)
-			)
-			(justify left bottom)
-		)
-	)
-	(text "14. CONDENSADORES (2026-09-28): 100 nF fora do 24 V ="
-		(exclude_from_sim no)
-		(at 22.86 129.54 0)
-		(effects
-			(font
-				(size 1.27 1.27)
-			)
-			(justify left bottom)
-		)
-	)
-	(text "    TDK C1608X7R1H104K080AA (X7R 50 V, catalogo TDK p.34)."
-		(exclude_from_sim no)
-		(at 22.86 133.35 0)
-		(effects
-			(font
-				(size 1.27 1.27)
-			)
-			(justify left bottom)
-		)
-	)
-	(text "    Pior caso fora do 24 V: +12V_TPS a 31,7 V (folha 6,"
-		(exclude_from_sim no)
-		(at 22.86 137.16 0)
-		(effects
-			(font
-				(size 1.27 1.27)
-			)
-			(justify left bottom)
-		)
-	)
-	(text "    nota 17), por isso 50 V e nao 25 V. C36 (+24V_ADC,"
-		(exclude_from_sim no)
-		(at 22.86 140.97 0)
-		(effects
-			(font
-				(size 1.27 1.27)
-			)
-			(justify left bottom)
-		)
-	)
-	(text "    ate 53,3 V) fica GRM188R72A104KA35D 100 V."
-		(exclude_from_sim no)
-		(at 22.86 144.78 0)
-		(effects
-			(font
-				(size 1.27 1.27)
-			)
-			(justify left bottom)
-		)
-	)
-	(text "    1 uF = TDK C1608X7R1H105K080AB (X7R 50 V, p.35) nos 4."
-		(exclude_from_sim no)
-		(at 22.86 148.58999999999997 0)
-		(effects
-			(font
-				(size 1.27 1.27)
-			)
-			(justify left bottom)
-		)
-	)

Commit message: Limpeza do ERC/DRC: fio solto e rotulo duplicado na folha 5, notas do C1 na folha 2, texto do C35
- 05_adc: removido o troco de fio de 1,27 mm em (128,27; 78,74)-(128,27; 80,01)
  com a junction que so existia por ele (extremo sem ligacao no ERC), e o
  rotulo local +2.5_VREF sobreposto ao global em (236,22; 83,82).
- 02_entrada: notas 4 e 12 falavam de "C1/C13" da numeracao antiga; o C13 e
  hoje o bypass do VCC2 do U5. A entrada do U1 (R-78HB) e o C1.
- PCB: texto de serigrafia ${REFERENCE} do C35 afastado do pad do C36.

Netlist do kicad-cli identica pino a pino antes/depois (104 redes;
+2.5_VREF = C24, C25, R8, U6.20, U7.6). DRC com paridade: 0 erros, 0 avisos,
0 desligados, paridade 0. Pacote de fabricacao regenerado.

Co-Authored-By: Claude Opus 5.5 (1M context) <noreply@anthropic.com>
Claude-Session: https://claude.ai/code/session_01KPnkiJQKrkjgRqqw9M78ie
Other:
- note added: "12. C1 = GRM32EC72A106KE05 (1210 X7S 10 uF 100 V,"
- note added: "4. C1 = 10 uF a 100 V: o clamp de 53,3 V fica acima de"
- note added: "C1 retorna a GND_ADC = GND do U1. (C13 e hoje o bypass do U5.)"
- note added: "Murata cat. 2021 p.110). Com o U1 = R-78HB, o C1 e a"
- note added: "entrada junto ao Vin (PCB 28-09: 2,9 mm do pino 1); massa"
- note removed: "10 uF/100 V ceramico junto ao Vin (C13); C1 e o bulk"
- note removed: "12. C1/C13 = GRM32EC72A106KE05 (1210 X7S 10 uF 100 V,"
- note removed: "4. C1/C13 = 10 uF a 100 V: o clamp de 53,3 V fica acima de"
- note removed: "C13 retorna a GND_ADC = GND do modulo (Fig. 5)."
- note removed: "Murata cat. 2021 p.110): MORNSUN Tab.1 p.3 pede C1 ="
Changed lines of the file:
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@@
 		)
 	)
-	(text "    Murata cat. 2021 p.110): MORNSUN Tab.1 p.3 pede C1 ="
+	(text "    Murata cat. 2021 p.110). Com o U1 = R-78HB, o C1 e a"
 		(exclude_from_sim no)
 		(at 114.3 171.45 0)
@@
 		)
 	)
-	(text "12. C1/C13 = GRM32EC72A106KE05 (1210 X7S 10 uF 100 V,"
+	(text "12. C1 = GRM32EC72A106KE05 (1210 X7S 10 uF 100 V,"
 		(exclude_from_sim no)
 		(at 114.3 167.64 0)
@@
 		)
 	)
-	(text "4. C1/C13 = 10 uF a 100 V: o clamp de 53,3 V fica acima de"
+	(text "4. C1 = 10 uF a 100 V: o clamp de 53,3 V fica acima de"
 		(exclude_from_sim no)
 		(at 114.3 83.82 0)
@@
 		)
 	)
-	(text "    C13 retorna a GND_ADC = GND do modulo (Fig. 5)."
+	(text "    C1 retorna a GND_ADC = GND do U1. (C13 e hoje o bypass do U5.)"
 		(exclude_from_sim no)
 		(at 114.3 182.88 0)
@@
 		)
 	)
-	(text "    10 uF/100 V ceramico junto ao Vin (C13); C1 e o bulk"
+	(text "    entrada junto ao Vin (PCB 28-09: 2,9 mm do pino 1); massa"
 		(exclude_from_sim no)
 		(at 114.3 175.26 0)
