File: Desenvolvimento_IC2S-EBM7-2608-V2.3-Fixo420/Projeto_IC2S-EBM7-2608-V2.3-Fixo420/06_lacos.kicad_sch (KiCad schematic)
At the start: 58 parts, among them T8 TP_+24V_ADC, U10 TPS26613DDFR, U11 TPS26613DDFR, U12 TPS7A4001DGN, U8 TPS26613DDFR, U9 TPS26613DDFR

Commit message: Roteamento do U2 (SPX3819) e do bypass do ISO7141; pacote de fabricacao regenerado
PCB:
- C49 (2,2 uF) e C8 (10 uF) junto do VOUT do U2 (1,68 e 2,23 mm), C6 na
  entrada a 3,0 mm.
- C9 (100 nF) reposto como bypass do VCC1 do U5 (1,93 mm), massa por via
  DGND a 1,0 mm do pad. Tinha sido movido com o grupo do U2 (6,3 mm).
- Rede unconnected-(U2-BP-Pad4) na classe DIGSIDE (pad NC do SPX3819 dentro
  da zona DGND; sem isto a regra de barreira de 1,0 mm disparava contra C9).
- DRC kicad-cli com paridade: 0 erros, 0 avisos, 0 desligados, paridade 0.

Esquematico: sem alteracao electrica (paridade 0, netlist igual). Restauro do
historico local do KiCad: coordenadas arredondadas (02), fios colineares
fundidos com os mesmos extremos (04), rectangulo grafico removido (06),
ordem dos textos (08).

Fabricacao: Gerbers, furacao, PnP, stencil, BOM, vistas, STEP e PDF do
esquematico regenerados desta placa (antes eram de 28-09 02:48).

Co-Authored-By: Claude Opus 5.5 (1M context) <noreply@anthropic.com>
Claude-Session: https://claude.ai/code/session_01KPnkiJQKrkjgRqqw9M78ie
Changed lines of the file:
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@@
-	)
-	(rectangle
-		(start 208.28 179.07)
-		(end 265.43 204.47)
-		(stroke
-			(width 0)
-			(type default)
-		)
-		(fill
-			(type none)
-		)
 	)
 	(rectangle

Commit message: Lacos 4-20 mA: limitador discreto no lugar dos TPS26613 e do TPS7A4001
Folha 6: saem U8-U11 (TPS26613), U12 (TPS7A4001), o +12V_TPS, o divisor VSNS
(R22-R26) e C26/C29/C31/C32/C37/C38. Por laco entra um limitador discreto:
Q1-Q4 BSP297 (D no AINk, S -> R40-R43 18R -> burden), Q5-Q8 BC847C com B/E sobre
o 18R e C na porta; porta por R44-R47 100k desde VZ_LIM = +24V_ADC -> R48 22k ->
D26 BZT52H-C10 (C50 100n). D6/D7/D8/D11 passam a SMBJ36A e as burden R13-R15/R17
a TNPW1206 0,1 %.

Pinagens conferidas no desenho das folhas (BSP297 Rev.2.2 p.1, BC847X Rev.13 p.2,
BZT52H Rev.7 p.2). Simbolos novos em EBM7_V23_proyecto11; footprint
SOT-223-3_TabPin2 (aba = dreno).

Portas: netlist com a particao dos pinos nao tocados identica (94 grupos) e as
redes novas com os membros exactos, ERC 0 erros. Simulacao ngspice com modelos
Infineon/Nexperia: limite 23,7-39 mA de -40 a 85 C, compliance -0,38 V a 20 mA,
surto 1 kV com 0,017/0,094 mJ na burden.

A PCB NAO foi actualizada. Pendente: cobre para RthJA <= ~90 K/W em cada Q1-Q4,
ensaio de bancada e revisao independente. Ver
alteracao_limitador_discreto_lacos_2026-10-02.md.

Co-Authored-By: Claude Opus 5.5 (1M context) <noreply@anthropic.com>
Parts:
- removed C26, C29, C31, C32, C37: 100nF/50V, EBM7_V23:0603C, symbol Device:C
- removed C38: 10uF/50V, EBM7_V23:C_1206_3216Metric, symbol Device:C
- removed R22: 11k5, EBM7_V23:0603R, symbol Device:R
- removed R23, R24: 6k65, EBM7_V23:0603R, symbol Device:R
- removed R25: 93k1, EBM7_V23:0603R, symbol Device:R
- removed R26: 10k, EBM7_V23:0603R, symbol Device:R
- removed U10, U11, U8, U9: TPS26613DDFR, EBM7_V23:SOT-23-8, symbol EBM7_V23_proyecto7:TPS26613DDFR
- removed U12: TPS7A4001DGN, EBM7_V23:HVSSOP-8-1EP, symbol EBM7_V23_proyecto9:TPS7A4001DGN
- added C50: 100nF/50V, EBM7_V23:0603C, symbol Device:C
- added D26: BZT52H-C10, EBM7_V23:SOD-123F, symbol Device:D_Zener
- added Q1, Q2, Q3, Q4: BSP297, EBM7_V23:SOT-223-3_TabPin2, symbol EBM7_V23_proyecto11:BSP297
- added Q5, Q6, Q7, Q8: BC847C, EBM7_V23:SOT-23, symbol EBM7_V23_proyecto11:BC847C
- added R40, R41, R42, R43: 18R, EBM7_V23:0603R, symbol Device:R
- added R44, R45, R46, R47: 100k, EBM7_V23:0603R, symbol Device:R
- added R48: 22k, EBM7_V23:0603R, symbol Device:R
- D11, D6, D7, D8: value 824500301 -> SMBJ36A; footprint EBM7_V23:DO-214 -> EBM7_V23:DO-214AA; MPN 824500301 -> SMBJ36A-13-F
- R13, R14, R15, R17: footprint EBM7_V23:0603R -> EBM7_V23:1206R; MPN RG1608P-111-B-T5 -> TNPW1206110RBEEA
Connections:
- net +24V_ADC: now also R48.1
- net AIN1: now also Q1.2 (D)
- net AIN2: now also Q2.2 (D)
- net AIN3: now also Q3.2 (D)
- net AIN4: now also Q4.2 (D)
- net GND_ADC: now also C50.2, D26.2 (A)
- net at R11.2: now also Q6.2 (E), R41.1
- net at R10.2: now also Q5.2 (E), R40.1
- net at R12.2: now also Q7.2 (E), R42.1
- net at R16.2: now also Q8.2 (E), R43.1
- new net: Q1.3 (S), Q5.1 (B), R40.2
- new net: Q4.3 (S), Q8.1 (B), R43.2
- new net: Q2.3 (S), Q6.1 (B), R41.2
- new net: Q3.3 (S), Q7.1 (B), R42.2
- new net LIM1_G: Q1.1 (G), Q5.3 (C), R44.1
- new net LIM2_G: Q2.1 (G), Q6.3 (C), R45.1
- new net LIM3_G: Q3.1 (G), Q7.3 (C), R46.1
- new net LIM4_G: Q4.1 (G), Q8.3 (C), R47.1
- new net VZ_LIM: C50.1, D26.1 (K), R44.2, R45.2, R46.2, R47.2, R48.2
- no-connect marks 4 -> 0
Other:
- note added: "(C50 100n). O zener faz o papel do +Vs do TPS: o no da burden fica <= ~8,5 V"
- note added: "(falam do TPS26613 e do TPS7A4001)."
- note added: "(rama lacos-limitador-discreto). Retirados U8-U11 TPS26613, U12 TPS7A4001,"
- note added: "+12V_TPS, VSNS, R22-R26, C26, C29, C31, C32, C37 e C38."
- note added: "85 C (ngspice, modelos Infineon BSP297_L0 e Nexperia BC847C; bancada: falta)."
- note added: "D6/D7/D8/D11 -> SMBJ36A: numa falha a linha AIN fica no +24V_AIN (>= 36 V)."
- note added: "DECISAO 2026-10-02 - limitador discreto nos lacos"
- note added: "Firmware: leitura >= 21 mA (NAMUR NE43) = falha ou curto no laco."
- note added: "Notas 1, 5, 8-11, 16 e o cabecalho DECISAO 21-09-2026 ficam HISTORICAS"
- note added: "Por laco: Q1-Q4 BSP297 (D no AINk) -> R40-R43 18R -> burden. Q5-Q8 BC847C"
- note added: "Porta: R44-R47 100k desde VZ_LIM = +24V_ADC -> R48 22k -> D26 BZT52H-C10"
- note added: "Q1-Q4 cobre para RthJA <= ~90 K/W (6 cm2 = 70 K/W; BSP297 Rev.2.2 p.2)."
- note added: "Q5-Q8 longe de Q1-Q4 (aquecidos juntos, I_lim desce abaixo de 21 mA)."
- note added: "R13-R15/R17 -> TNPW1206 0,1% 25ppm: ate 169 mW (0603 de 0,1 W nao chega)."
- note added: "Sem corte termico: Q1-Q4 dissipam 0,67-1,06 W numa falha mantida a 32 V."
- note added: "Tj = Ta + P x RthJA: com pegada minima (115 K/W) da 162 C a 85 C. Dar a cada"
- note added: "com B/E sobre os 18R e C na porta: I_lim = VBE/18R = 23,7-39 mA de -40 a"
- note added: "mesmo com a burden aberta (1,4 mA para o ADC)."
